File: Hardware/PTH/SparkFun_BlueSMiRF-v2-Headers.kicad_sch (KiCad schematic)
At the start: 38 parts, among them J1 Conn_01x06, Q1 Q_NMOS_DGS, Q2 Q_NMOS_DGS, SW1 Switch, U1 ESP32_Pico_Mini, U2 AP2112K-3.3

Commit message: Rename to BlueSMiRF v2.
Other:
- title: SparkFun BlueSMiRF - ESP32 PTH -> SparkFun BlueSMiRF v2 - Headers
Changed lines of the file:
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@@
   (paper "USLetter")
   (title_block
-    (title "SparkFun BlueSMiRF - ESP32 PTH")
+    (title "SparkFun BlueSMiRF v2 - Headers")
     (date "2023-07-29")
     (rev "v11")
