File: Hardware/SMD/SparkFun_BlueSMiRF-v2.kicad_pcb (KiCad board)
At the start: 2 copper layers, 38.1 x 15.2 mm, 57 parts, among them J1 Conn_01x06, Q1 NMOS_0.2A_50V, Q2 NMOS_0.2A_50V, SW1 SPST_Momentary_4.6x2.8mm, U1 ESP32-PICO-V3-02, U2 AP2112K-3.3

Commit message: Rename to BlueSMiRF v2.
Parts:
- moved U3 194.8 mm to (180.3, 81.3)
Changed lines of the file:
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@@
   )
   (footprint "SparkFun-Aesthetic:ORDERING_INSTRUCTIONS" (layer "F.Cu")
-    (at 1.52 4.06)
+    (at 180.34 81.28)
     (property "Sheetfile" "SparkFun_BlueSMiRF-ESP32.kicad_sch")
     (property "Sheetname" "")
