File: Hardware/SMD/SparkFun_BlueSMiRF-v2.kicad_sch (KiCad schematic)
At the start: 38 parts, among them J1 Conn_01x06, Q1 NMOS_0.2A_50V, Q2 NMOS_0.2A_50V, SW1 SPST_Momentary_4.6x2.8mm, U1 ESP32-PICO-V3-02, U2 AP2112K-3.3

Commit message: Rename to BlueSMiRF v2.
Other:
- title: SparkFun BlueSMiRF - ESP32 -> SparkFun BlueSMiRF v2
Changed lines of the file:
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@@
   (paper "USLetter")
   (title_block
-    (title "SparkFun BlueSMiRF - ESP32")
+    (title "SparkFun BlueSMiRF v2")
     (date "2023-07-29")
-    (rev "v10")
+    (rev "v11")
     (comment 1 "Designed by: N. Seidle")
   )
